Commit message: firmware tested and ros2 cad updates
Co-Authored-By: Claude Sonnet 5.5 <noreply@anthropic.com>

File: ros_ws/src/mini_tesla_description/urdf/mini_tesla.urdf.xacro (robot description, xacro)
@@ -1,5 +1,5 @@
 <?xml version="1.0"?>
 <!--
-  Mini Tesla 10C4I - indoor mecanum robot (FINAL rev 2 chassis)
+  Mini Tesla 10C4I - indoor mecanum robot (rev3 chassis)
   ROS 2 Jazzy + Gazebo Harmonic.
   Frames: base_footprint on the floor under the robot centre; base_link = chassis underside centre
@@ -8,12 +8,8 @@
     drive        mecanum (default): wheels driven by gz MecanumDrive with 45-degree friction
                  planar: ideal holonomic base (VelocityControl), wheels slide; use if contact tuning bites
-    side_radars  false (default) / true   radars on both side extensions
-    rear_radar   false (default) / true
     laptop       true (default) / false   ASUS G14 on the deck (1.5 kg)
 -->
 <robot name="mini_tesla" xmlns:xacro="http://www.ros.org/wiki/xacro" xmlns:gz="http://gazebosim.org/schema">
   <xacro:arg name="drive" default="mecanum"/>
-  <xacro:arg name="side_radars" default="false"/>
-  <xacro:arg name="rear_radar" default="false"/>
   <xacro:arg name="laptop" default="true"/>
   <xacro:property name="pkg" value="$(find mini_tesla_description)"/>
@@ -35,5 +31,4 @@
   <xacro:property name="m_laptop" value="1.50"/>
   <xacro:property name="m_wheel" value="0.12"/>          <!-- REV 75 mm mecanum + printed adapter -->
-  <xacro:property name="m_camera" value="0.061"/>
   <!-- motor: Pololu 37D 19:1 -> ~530 rpm no-load = 55 rad/s -->
   <xacro:property name="wheel_vel_limit" value="55.0"/>

File: ros_ws/src/mini_tesla_description/urdf/sensors.xacro (robot description, xacro)
@@ -7,14 +7,18 @@
                      scan into a sensor_msgs/Range (nearest beam), like the real sensor's single distance.
     IWR6843 radar -> gpu_lidar: 120 x 40 deg, 0.1-10 m, 10 Hz, published as a PointCloud2 (no Doppler).
-    OAK-D Lite    -> rgbd_camera 640x480 @ 30 Hz (73 deg HFOV) + its BMI270 IMU @ 200 Hz.
+    iPhone 16 Pro -> rgbd_camera 640x480 @ 30 Hz on the 24 mm main camera (HFOV 71.4 deg: 24 mm is the
+                     35 mm-equivalent focal length Apple publishes; Apple does not publish the FOV itself),
+                     depth out to 5 m (Apple: LiDAR Scanner works up to 5 m), IMU @ 100 Hz.
+    Velodyne Puck LITE -> gpu_lidar from the datasheet: 16 ch, +-15 deg (2 deg steps), 360 deg x 0.2 deg,
+                     10 Hz, 0.5-100 m, +-3 cm. Published as a PointCloud2.
 -->
 <robot xmlns:xacro="http://www.ros.org/wiki/xacro">
-  <xacro:property name="sensor_z" value="0.023"/>   <!-- all ToF + radar centres, 44 mm above the floor -->
+  <xacro:property name="sensor_z" value="0.023"/>   <!-- ToF + radar centres, 44 mm above the floor -->
   <!-- ===================== VL53L1X ToF ===================== -->
-  <xacro:macro name="tof" params="name x y yaw">
+  <xacro:macro name="tof" params="name x y yaw z:=${sensor_z}">
     <joint name="tof_${name}_joint" type="fixed">
       <parent link="base_link"/>
       <child link="tof_${name}_link"/>
-      <origin xyz="${x} ${y} ${sensor_z}" rpy="0 0 ${yaw}"/>
+      <origin xyz="${x} ${y} ${z}" rpy="0 0 ${yaw}"/>
     </joint>
     <link name="tof_${name}_link"/>
@@ -55,14 +59,14 @@
     </gazebo>
   </xacro:macro>
-  <!-- bumpers: front and rear pairs at y = +-84 mm, board face 184 mm from centre -->
-  <xacro:tof name="front_left"  x="0.18415"  y="0.084"   yaw="0"/>
-  <xacro:tof name="front_right" x="0.18415"  y="-0.084"  yaw="0"/>
-  <xacro:tof name="rear_left"   x="-0.18415" y="0.084"   yaw="${pi}"/>
-  <xacro:tof name="rear_right"  x="-0.18415" y="-0.084"  yaw="${pi}"/>
-  <!-- side extensions: x = +-78 mm, board face at y = +-145.6 mm -->
-  <xacro:tof name="left_front"  x="0.078"    y="0.1456"  yaw="${pi/2}"/>
-  <xacro:tof name="left_rear"   x="-0.078"   y="0.1456"  yaw="${pi/2}"/>
-  <xacro:tof name="right_front" x="0.078"    y="-0.1456" yaw="${-pi/2}"/>
-  <xacro:tof name="right_rear"  x="-0.078"   y="-0.1456" yaw="${-pi/2}"/>
+  <!-- rev3: four pods on the faces (front one is raised onto the phone-mount side, z 62 mm) and four
+       45 deg corner boards. Positions are the CAD board centres. -->
+  <xacro:tof name="front"       x="0.1938"  y="0"       yaw="0"        z="0.062"/>
+  <xacro:tof name="rear"        x="-0.1948" y="0"       yaw="${pi}"/>
+  <xacro:tof name="left"        x="0"       y="0.1463"  yaw="${pi/2}"/>
+  <xacro:tof name="right"       x="0"       y="-0.1463" yaw="${-pi/2}"/>
+  <xacro:tof name="front_left"  x="0.197"   y="0.086"   yaw="${pi/4}"/>
+  <xacro:tof name="front_right" x="0.197"   y="-0.086"  yaw="${-pi/4}"/>
+  <xacro:tof name="rear_left"   x="-0.197"  y="0.086"   yaw="${3*pi/4}"/>
+  <xacro:tof name="rear_right"  x="-0.197"  y="-0.086"  yaw="${-3*pi/4}"/>
   <!-- ===================== TI IWR6843AOPEVM radar ===================== -->
   <xacro:macro name="radar" params="name x y yaw">
@@ -109,54 +113,55 @@
     </gazebo>
   </xacro:macro>
-  <!-- front: antenna (chip) centre on the bumper -->
+  <!-- front: antenna (chip) centre on the front bumper -->
   <xacro:radar name="front" x="0.1920" y="-0.0201" yaw="0"/>
-  <xacro:if value="$(arg side_radars)">
-    <xacro:radar name="left"  x="0.0233"  y="0.15345"  yaw="${pi/2}"/>
-    <xacro:radar name="right" x="-0.0233" y="-0.15345" yaw="${-pi/2}"/>
-  </xacro:if>
-  <xacro:if value="$(arg rear_radar)">
-    <xacro:radar name="rear" x="-0.1920" y="0.0201" yaw="${pi}"/>
-  </xacro:if>
-  <!-- ===================== OAK-D Lite ===================== -->
-  <!-- camera_link = centre of the camera's front face (x 188 mm, z 75 mm above the chassis underside) -->
-  <joint name="oak_joint" type="fixed">
+  <!-- ===================== iPhone 16 Pro (front phone mount) ===================== -->
+  <!-- iphone_link = centre of the phone body (CAD x 179.1, z 112.8 mm). The camera bump faces +X; the
+       main camera / LiDAR scanner sit at y +50 mm, z +11 mm of the body centre, 6.4 mm in front of it. -->
+  <xacro:property name="m_phone" value="0.199"/>
+  <joint name="iphone_joint" type="fixed">
     <parent link="base_link"/>
-    <child link="oak_link"/>
-    <origin xyz="0.188 0 0.075" rpy="0 0 0"/>
-  </joint>
-  <link name="oak_link">
+    <child link="iphone_link"/>
+    <origin xyz="0.1791 0 0.1128" rpy="0 0 0"/>
+  </joint>
+  <link name="iphone_link">
     <visual>
-      <geometry><mesh filename="file://${pkg}/meshes/oak_d_lite.stl" scale="${mesh_scale}"/></geometry>
+      <geometry><mesh filename="file://${pkg}/meshes/iphone.stl" scale="${mesh_scale}"/></geometry>
       <material name="black"/>
     </visual>
     <collision>
-      <origin xyz="-0.00875 0 0" rpy="0 0 0"/>
-      <geometry><box size="0.0175 0.091 0.028"/></geometry>
+      <origin xyz="-0.002 0 0" rpy="0 0 0"/>
+      <geometry><box size="0.0126 0.1496 0.0715"/></geometry>
     </collision>
-    <xacro:box_inertial m="${m_camera}" x="0.0175" y="0.091" z="0.028">
-      <origin xyz="-0.00875 0 0" rpy="0 0 0"/>
+    <xacro:box_inertial m="${m_phone}" x="0.0083" y="0.1496" z="0.0715">
+      <origin xyz="-0.002 0 0" rpy="0 0 0"/>
     </xacro:box_inertial>
   </link>
-  <joint name="oak_optical_joint" type="fixed">
-    <parent link="oak_link"/>
-    <child link="oak_optical_frame"/>
+  <joint name="iphone_camera_joint" type="fixed">
+    <parent link="iphone_link"/>
+    <child link="iphone_camera_link"/>
+    <origin xyz="0.0064 0.050 0.011" rpy="0 0 0"/>
+  </joint>
+  <link name="iphone_camera_link"/>
+  <joint name="iphone_optical_joint" type="fixed">
+    <parent link="iphone_camera_link"/>
+    <child link="iphone_optical_frame"/>
     <origin xyz="0 0 0" rpy="${-pi/2} 0 ${-pi/2}"/>
   </joint>
-  <link name="oak_optical_frame"/>
-  <joint name="oak_imu_joint" type="fixed">
-    <parent link="oak_link"/>
-    <child link="oak_imu_link"/>
-    <origin xyz="-0.009 0 0" rpy="0 0 0"/>
-  </joint>
-  <link name="oak_imu_link"/>
-  <gazebo reference="oak_link">
-    <sensor name="oak_rgbd" type="rgbd_camera">
-      <gz_frame_id>oak_optical_frame</gz_frame_id>
-      <topic>/oak/rgbd</topic>
+  <link name="iphone_optical_frame"/>
+  <joint name="iphone_imu_joint" type="fixed">
+    <parent link="iphone_link"/>
+    <child link="iphone_imu_link"/>
+    <origin xyz="0 0 0" rpy="0 0 0"/>
+  </joint>
+  <link name="iphone_imu_link"/>
+  <gazebo reference="iphone_camera_link">
+    <sensor name="iphone_rgbd" type="rgbd_camera">
+      <gz_frame_id>iphone_optical_frame</gz_frame_id>
+      <topic>/iphone/rgbd</topic>
       <update_rate>30</update_rate>
       <always_on>true</always_on>
       <visualize>true</visualize>
       <camera>
-        <horizontal_fov>1.274</horizontal_fov>
+        <horizontal_fov>1.246</horizontal_fov>
         <image>
           <width>640</width>
@@ -171,5 +176,5 @@
           <clip>
             <near>0.20</near>
-            <far>10.0</far>
+            <far>5.0</far>
           </clip>
         </depth_camera>
@@ -182,9 +187,9 @@
     </sensor>
   </gazebo>
-  <gazebo reference="oak_imu_link">
-    <sensor name="oak_imu" type="imu">
-      <gz_frame_id>oak_imu_link</gz_frame_id>
-      <topic>/oak/imu</topic>
-      <update_rate>200</update_rate>
+  <gazebo reference="iphone_imu_link">
+    <sensor name="iphone_imu" type="imu">
+      <gz_frame_id>iphone_imu_link</gz_frame_id>
+      <topic>/iphone/imu</topic>
+      <update_rate>100</update_rate>
       <always_on>true</always_on>
       <imu>
@@ -202,3 +207,70 @@
     </sensor>
   </gazebo>
+  <!-- ===================== Velodyne Puck LITE on the rear mast ===================== -->
+  <!-- velodyne_base_link = bottom of the puck (CAD x -192 mm, z 272 mm); the scan origin is 37.7 mm above it
+       (Puck LITE datasheet: optical centre 37.8 mm). The mast itself is part of the mounts mesh. -->
+  <xacro:property name="m_velodyne" value="0.59"/>
+  <joint name="velodyne_base_joint" type="fixed">
+    <parent link="base_link"/>
+    <child link="velodyne_base_link"/>
+    <origin xyz="-0.192 0 0.272" rpy="0 0 0"/>
+  </joint>
+  <link name="velodyne_base_link">
+    <visual>
+      <geometry><mesh filename="file://${pkg}/meshes/velodyne_puck.stl" scale="${mesh_scale}"/></geometry>
+      <material name="black"/>
+    </visual>
+    <collision>
+      <origin xyz="0 0 0.03585" rpy="0 0 0"/>
+      <geometry><cylinder radius="0.05165" length="0.0717"/></geometry>
+    </collision>
+    <inertial>
+      <origin xyz="0 0 0.03585" rpy="0 0 0"/>
+      <mass value="${m_velodyne}"/>
+      <inertia ixx="${m_velodyne*(3*0.05165*0.05165+0.0717*0.0717)/12}" ixy="0" ixz="0"
+               iyy="${m_velodyne*(3*0.05165*0.05165+0.0717*0.0717)/12}" iyz="0"
+               izz="${m_velodyne*0.05165*0.05165/2}"/>
+    </inertial>
+  </link>
+  <joint name="velodyne_joint" type="fixed">
+    <parent link="velodyne_base_link"/>
+    <child link="velodyne"/>
+    <origin xyz="0 0 0.0378" rpy="0 0 0"/>
+  </joint>
+  <link name="velodyne"/>
+  <gazebo reference="velodyne">
+    <sensor name="velodyne" type="gpu_lidar">
+      <gz_frame_id>velodyne</gz_frame_id>
+      <topic>/velodyne/scan</topic>
+      <update_rate>10</update_rate>
+      <always_on>true</always_on>
+      <visualize>false</visualize>
+      <lidar>
+        <scan>
+          <horizontal>
+            <samples>1800</samples>
+            <resolution>1</resolution>
+            <min_angle>-3.14159</min_angle>
+            <max_angle>3.14159</max_angle>
+          </horizontal>
+          <vertical>
+            <samples>16</samples>
+            <resolution>1</resolution>
+            <min_angle>-0.2618</min_angle>
+            <max_angle>0.2618</max_angle>
+          </vertical>
+        </scan>
+        <range>
+          <min>0.5</min>
+          <max>100.0</max>
+          <resolution>0.003</resolution>
+        </range>
+        <noise>
+          <type>gaussian</type>
+          <mean>0.0</mean>
+          <stddev>0.03</stddev>
+        </noise>
+      </lidar>
+    </sensor>
+  </gazebo>
 </robot>
